Commit message: Gazebo jala, ROS2 No

File: tm_empl1_description/urdf/basic_link_position.xacro (robot description, xacro)
@@ -5,6 +5,8 @@
     <link name="world">
     </link>
-    <joint name="world_to_baselink" type="fix">
-        <origin xyz="0 0 0.15" rpy="0 0 0"/>
+    <joint name="world_to_baselink" type="fixed">
+        <parent link="world" />
+        <child link="base_link" />
+        <origin xyz="0 0 0" rpy="0 0 0"/>
     </joint>
     <link name="base_link">
